Commit message: fix frame tf

File: catkin_ws/src/husky_description/urdf/accessories/camera.urdf.xacro (robot description, xacro)
@@ -43,8 +43,14 @@
       </collision>
     </link>
-    <joint name="${parent}_optical_joint" type="fixed">
+    <joint name="${parent}_camera_link_joint" type="fixed">
       <xacro:insert_block name="origin"/>
       <parent link="${parent}"/>
       <child link="${name}_link"/>
+    </joint>
+    <link name="${name}"/>
+    <joint name="${parent}_camera_joint" type="fixed">
+      <origin xyz="0 0 0" rpy="-1.57 0 -1.57"/>
+      <parent link="${name}_link"/>
+      <child link="${name}"/>
     </joint>
     <gazebo reference="${name}_link">
